File: presTimer.sch (EAGLE design)
At the start: 9 parts, among them J2 POWER_JACKPTH

Commit message: Updated circuit board layout
Changed lines of the file:
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@@
 <wire x1="106.68" y1="78.74" x2="88.9" y2="66.04" width="0.1524" layer="91"/>
 <junction x="88.9" y="66.04"/>
+<wire x1="106.68" y1="78.74" x2="106.68" y2="63.5" width="0.1524" layer="91"/>
+<junction x="106.68" y="78.74"/>
+<wire x1="106.68" y1="63.5" x2="88.9" y2="63.5" width="0.1524" layer="91"/>
+<wire x1="88.9" y1="63.5" x2="88.9" y2="66.04" width="0.1524" layer="91"/>
 </segment>
 </net>
